File: hardware/wled_controller/drivers.kicad_sch (KiCad schematic)
At the start: 12 parts, among them J1 Screw_Terminal_01x03, J10 Screw_Terminal_01x03, J11 Screw_Terminal_01x03, J12 Screw_Terminal_01x03, J2 Screw_Terminal_01x03, J3 Screw_Terminal_01x03, J4 Screw_Terminal_01x03, J5 Screw_Terminal_01x03, J6 Screw_Terminal_01x03, J7 Screw_Terminal_01x03, J8 Screw_Terminal_01x03, J9 Screw_Terminal_01x03

Commit message: finalise schematic
Parts:
- added J13, J14, J15: Screw_Terminal_01x03, conn:TerminalBlock_4Ucon_1x03_P3.50mm_Vertical, symbol conn:Screw_Terminal_01x03
Connections:
- net GND: now also J13.3 (Pin_3), J14.3 (Pin_3), J15.3 (Pin_3)
- net VDD: now also J13.1 (Pin_1), J14.1 (Pin_1), J15.1 (Pin_1)
- new net WLED driver 13/DOUT: J13.2 (Pin_2)
- new net WLED driver 14/DOUT: J14.2 (Pin_2)
- new net WLED driver 15/DOUT: J15.2 (Pin_2)
Other:
- added sheet WLED driver 13 (wled_driver.kicad_sch)
- added sheet WLED driver 14 (wled_driver.kicad_sch)
- added sheet WLED driver 15 (wled_driver.kicad_sch)
- moved on the sheet: J1, J10, J11, J12, J2, J3, J4, J5, J6, J7, J8, J9

Commit message: some progress on PCB
Parts:
- J1: footprint conn:TerminalBlock_4Ucon_1x03_P3.50mm_Vertical -> conn:TerminalBlock_Degson_1x03_P3.50mm_Horizontal; Part 15EDGVC-3.5-03P-14-00Z(H), 15EDGKA-3.5-03P-14-100AH -> 15EDGRC-3.5-03P-14-00AH, 15EDGKA-3.5-03P-14-100AH; Shop https://store.comet.bg/Catalogue/Product/45041/, https://st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 -> https://store.comet.bg/Catalogue/Product/45034/, https://st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
- J10, J11, J12, J13, J14, J15, J2, J3, J4, J5, J6, J7, J8, J9: footprint conn:TerminalBlock_4Ucon_1x03_P3.50mm_Vertical -> conn:TerminalBlock_Degson_1x03_P3.50mm_Horizontal
Connections:
- net WLED driver 10/DOUT: now also J5.2 (Pin_2); no longer J10.2 (Pin_2)
- net WLED driver 11/DOUT: now also J8.2 (Pin_2); no longer J11.2 (Pin_2)
- net WLED driver 12/DOUT: now also J10.2 (Pin_2); no longer J12.2 (Pin_2)
- net WLED driver 13/DOUT: now also J15.2 (Pin_2); no longer J13.2 (Pin_2)
- net WLED driver 15/DOUT: now also J12.2 (Pin_2); no longer J15.2 (Pin_2)
- net WLED driver 4/DOUT: now also J9.2 (Pin_2); no longer J4.2 (Pin_2)
- net WLED driver 5/DOUT: now also J11.2 (Pin_2); no longer J5.2 (Pin_2)
- net WLED driver 6/DOUT: now also J13.2 (Pin_2); no longer J6.2 (Pin_2)
- net WLED driver 7/DOUT: now also J4.2 (Pin_2); no longer J7.2 (Pin_2)
- net WLED driver 8/DOUT: now also J7.2 (Pin_2); no longer J8.2 (Pin_2)
- net WLED driver 9/DOUT: now also J6.2 (Pin_2); no longer J9.2 (Pin_2)

Commit message: work on pcb
Parts:
- J1: Part 15EDGRC-3.5-03P-14-00AH, 15EDGKA-3.5-03P-14-100AH -> 15EDGRC-3.5-03P-14-00AH, 15EDGK-3.5-03P-14-00AH; Shop https://store.comet.bg/Catalogue/Product/45034/, https://st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 -> https://store.comet.bg/Catalogue/Product/45034/
- J10, J11, J12, J13, J14, J15, J2, J3, J4, J5, J6, J7, J8, J9: Part 15EDGVC-3.5-03P-14-00Z(H), 15EDGKA-3.5-03P-14-100AH -> 15EDGRC-3.5-03P-14-00AH, 15EDGK-3.5-03P-14-00AH; Shop https://store.comet.bg/Catalogue/Product/45041/, https://st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 -> https://store.comet.bg/Catalogue/Product/45034/
