File: hardware/wled_controller/power_supply.kicad_sch (KiCad schematic)
At the start: 10 parts, among them J13 Screw_Terminal_01x02, U5 LMR54410

Commit message: finalise schematic
Parts:
- R13: Part R 118k 125mW 1% 0805 -> R 118kΩ 125mW 1% 0805
- U5: Part (none) -> LMR54410FDBVR; Shop (none) -> https://eu.mouser.com/ProductDetail/Texas-Instruments/LMR54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
- renumbered J13 to J16
Changed lines of the file:
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@@
 		(dnp no)
 		(fields_autoplaced yes)
-		(property "Reference" "#PWR064"
+		(property "Reference" "#PWR070"
 			(at 100.33 115.57 0)
 			(effects
@@
 			(project "wled_controller"
 				(path "/67a034fd-c582-46b2-83e2-3de9f5f70ac4/07b1b39b-eaae-4ce9-8e52-afae0c59cf87"
-					(reference "#PWR064")
+					(reference "#PWR070")
 					(unit 1)
 				)
@@
 			)
 		)
-		(property "Part" "R 118k 125mW 1% 0805"
+		(property "Part" "R 118kΩ 125mW 1% 0805"
 			(at 160.02 93.98 0)
 			(effects
@@
 		(dnp no)
 		(fields_autoplaced yes)
-		(property "Reference" "#PWR070"
+		(property "Reference" "#PWR076"
 			(at 195.58 115.57 0)
 			(effects
@@
 			(project "wled_controller"
 				(path "/67a034fd-c582-46b2-83e2-3de9f5f70ac4/07b1b39b-eaae-4ce9-8e52-afae0c59cf87"
-					(reference "#PWR070")
+					(reference "#PWR076")
 					(unit 1)
 				)
@@
 		(on_board yes)
 		(dnp no)
-		(property "Reference" "#PWR069"
+		(property "Reference" "#PWR075"
 			(at 195.58 86.36 0)
 			(effects
@@
 			(project "wled_controller"
 				(path "/67a034fd-c582-46b2-83e2-3de9f5f70ac4/07b1b39b-eaae-4ce9-8e52-afae0c59cf87"
-					(reference "#PWR069")
+					(reference "#PWR075")
 					(unit 1)
 				)
@@
 		(dnp no)
 		(fields_autoplaced yes)
-		(property "Reference" "#PWR068"
+		(property "Reference" "#PWR074"
 			(at 180.34 115.57 0)
 			(effects
@@
 			(project "wled_controller"
 				(path "/67a034fd-c582-46b2-83e2-3de9f5f70ac4/07b1b39b-eaae-4ce9-8e52-afae0c59cf87"
-					(reference "#PWR068")
+					(reference "#PWR074")
 					(unit 1)
 				)
@@
 		(on_board yes)
 		(dnp no)
-		(property "Reference" "J13"
+		(property "Reference" "J16"
 			(at 69.85 85.09 0)
 			(effects
@@
 			(project "wled_controller"
 				(path "/67a034fd-c582-46b2-83e2-3de9f5f70ac4/07b1b39b-eaae-4ce9-8e52-afae0c59cf87"
-					(reference "J13")
+					(reference "J16")
 					(unit 1)
 				)
@@
 		(dnp no)
 		(fields_autoplaced yes)
-		(property "Reference" "#PWR065"
+		(property "Reference" "#PWR071"
 			(at 109.22 115.57 0)
 			(effects
@@
 			(project "wled_controller"
 				(path "/67a034fd-c582-46b2-83e2-3de9f5f70ac4/07b1b39b-eaae-4ce9-8e52-afae0c59cf87"
-					(reference "#PWR065")
+					(reference "#PWR071")
 					(unit 1)
 				)
@@
 		(dnp no)
 		(fields_autoplaced yes)
-		(property "Reference" "#PWR062"
+		(property "Reference" "#PWR068"
 			(at 90.17 115.57 0)
 			(effects
@@
 			(project "wled_controller"
 				(path "/67a034fd-c582-46b2-83e2-3de9f5f70ac4/07b1b39b-eaae-4ce9-8e52-afae0c59cf87"
-					(reference "#PWR062")
+					(reference "#PWR068")
 					(unit 1)
 				)
@@
 			)
 		)
+		(property "Part" "LMR54410FDBVR"
+			(at 125.73 87.63 0)
+			(effects
+				(font
+					(size 1.27 1.27)
+				)
+				(hide yes)
+			)
+		)
+		(property "Shop" "https://eu.mouser.com/ProductDetail/Texas-Instruments/LMR54410FDBVR?qs=rSMjJ%252B1ewcShbG4Q7wcNsA%3D%3D"
+			(at 125.73 87.63 0)
+			(effects
+				(font
+					(size 1.27 1.27)
+				)
+				(hide yes)
+			)
+		)
 		(pin "3"
 		)
@@
 		(dnp no)
 		(fields_autoplaced yes)
-		(property "Reference" "#PWR066"
+		(property "Reference" "#PWR072"
 			(at 125.73 104.14 0)
 			(effects
@@
 			(project "wled_controller"
 				(path "/67a034fd-c582-46b2-83e2-3de9f5f70ac4/07b1b39b-eaae-4ce9-8e52-afae0c59cf87"
-					(reference "#PWR066")
+					(reference "#PWR072")
 					(unit 1)
 				)
@@
 		(on_board yes)
 		(dnp no)
-		(property "Reference" "#PWR063"
+		(property "Reference" "#PWR069"
 			(at 100.33 86.36 0)
 			(effects
@@
 			(project "wled_controller"
 				(path "/67a034fd-c582-46b2-83e2-3de9f5f70ac4/07b1b39b-eaae-4ce9-8e52-afae0c59cf87"
-					(reference "#PWR063")
+					(reference "#PWR069")
 					(unit 1)
 				)
@@
 		(dnp no)
 		(fields_autoplaced yes)
-		(property "Reference" "#PWR067"
+		(property "Reference" "#PWR073"
 			(at 160.02 115.57 0)
 			(effects
@@
 			(project "wled_controller"
 				(path "/67a034fd-c582-46b2-83e2-3de9f5f70ac4/07b1b39b-eaae-4ce9-8e52-afae0c59cf87"
-					(reference "#PWR067")
-					(unit 1)
-				)
+					(reference "#PWR073")
+					(unit 1)
+				)

Commit message: some progress on PCB
Parts:
- added D2: S2A, Diode_SMD:D_SMB, symbol Diode:1N4007
- added F1: Fuse, conn:Fuseholder_FS002, symbol Device:Polyfuse
- J16: footprint conn:TerminalBlock_4Ucon_1x02_P3.50mm_Vertical -> conn:TerminalBlock_1x02_P5.00mm_Horizontal; Part 15EDGVC-3.5-02P-14-00AH, 15EDGKA-3.5-02P-14-100AH -> DG127-5.0-02P-14-00AH; Shop https://store.comet.bg/Catalogue/Product/45040/, https://st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 -> https://store.comet.bg/Catalogue/Product/49346/
- renumbered U5 to U6
Connections:
- net GND: now also J16.1 (Pin_1), D2.1 (K); no longer J16.2 (Pin_2)
- net VDD: now also D2.2 (A), F1.2; no longer J16.1 (Pin_1)
- new net: F1.1, J16.2 (Pin_2)
Other:
- moved on the sheet: J16

Commit message: work on pcb
Parts:
- J16: Shop https://store.comet.bg/Catalogue/Product/49346/ -> https://store.comet.bg/Catalogue/Product/49346/, https://st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
- renumbered C4 to C3, C5 to C4, C6 to C5, C7 to C6, C8 to C7
Connections:
- net GND: now also U6.2 (GND); no longer U6.1 (GND)
Changed lines of the file:
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@@
 		(dnp no)
 		(fields_autoplaced yes)
-		(property "Reference" "#PWR071"
+		(property "Reference" "#PWR070"
 			(at 100.33 115.57 0)
 			(effects
@@
 			(project "wled_controller"
 				(path "/67a034fd-c582-46b2-83e2-3de9f5f70ac4/07b1b39b-eaae-4ce9-8e52-afae0c59cf87"
-					(reference "#PWR071")
+					(reference "#PWR070")
 					(unit 1)
 				)
@@
 		(dnp no)
 		(fields_autoplaced yes)
-		(property "Reference" "#PWR077"
+		(property "Reference" "#PWR076"
 			(at 195.58 115.57 0)
 			(effects
@@
 			(project "wled_controller"
 				(path "/67a034fd-c582-46b2-83e2-3de9f5f70ac4/07b1b39b-eaae-4ce9-8e52-afae0c59cf87"
-					(reference "#PWR077")
+					(reference "#PWR076")
 					(unit 1)
 				)
@@
 		(on_board yes)
 		(dnp no)
-		(property "Reference" "C6"
+		(property "Reference" "C5"
 			(at 142.24 78.74 0)
 			(effects
@@
 			(project "wled_controller"
 				(path "/67a034fd-c582-46b2-83e2-3de9f5f70ac4/07b1b39b-eaae-4ce9-8e52-afae0c59cf87"
-					(reference "C6")
+					(reference "C5")
 					(unit 1)
 				)
@@
 		(on_board yes)
 		(dnp no)
-		(property "Reference" "C8"
+		(property "Reference" "C7"
 			(at 196.85 96.52 0)
 			(effects
@@
 			(project "wled_controller"
 				(path "/67a034fd-c582-46b2-83e2-3de9f5f70ac4/07b1b39b-eaae-4ce9-8e52-afae0c59cf87"
-					(reference "C8")
+					(reference "C7")
 					(unit 1)
 				)
@@
 		(on_board yes)
 		(dnp no)
-		(property "Reference" "#PWR076"
+		(property "Reference" "#PWR075"
 			(at 195.58 86.36 0)
 			(effects
@@
 			(project "wled_controller"
 				(path "/67a034fd-c582-46b2-83e2-3de9f5f70ac4/07b1b39b-eaae-4ce9-8e52-afae0c59cf87"
-					(reference "#PWR076")
+					(reference "#PWR075")
 					(unit 1)
 				)
@@
 		(dnp no)
 		(fields_autoplaced yes)
-		(property "Reference" "#PWR069"
+		(property "Reference" "#PWR068"
 			(at 87.63 115.57 0)
 			(effects
@@
 			(project "wled_controller"
 				(path "/67a034fd-c582-46b2-83e2-3de9f5f70ac4/07b1b39b-eaae-4ce9-8e52-afae0c59cf87"
-					(reference "#PWR069")
+					(reference "#PWR068")
 					(unit 1)
 				)
@@
 		(dnp no)
 		(fields_autoplaced yes)
-		(property "Reference" "#PWR075"
+		(property "Reference" "#PWR074"
 			(at 180.34 115.57 0)
 			(effects
@@
 			(project "wled_controller"
 				(path "/67a034fd-c582-46b2-83e2-3de9f5f70ac4/07b1b39b-eaae-4ce9-8e52-afae0c59cf87"
-					(reference "#PWR075")
+					(reference "#PWR074")
 					(unit 1)
 				)
@@
 			)
 		)
-		(property "Shop" "https://store.comet.bg/Catalogue/Product/49346/"
+		(property "Shop" "https://store.comet.bg/Catalogue/Product/49346/, https://store.comet.bg/Catalogue/Product/45022/"
 			(at 62.23 87.63 0)
 			(effects
@@
 		(on_board yes)
 		(dnp no)
-		(property "Reference" "C5"
+		(property "Reference" "C4"
 			(at 110.49 96.52 0)
 			(effects
@@
 			(project "wled_controller"
 				(path "/67a034fd-c582-46b2-83e2-3de9f5f70ac4/07b1b39b-eaae-4ce9-8e52-afae0c59cf87"
-					(reference "C5")
+					(reference "C4")
 					(unit 1)
 				)
@@
 		(on_board yes)
 		(dnp no)
-		(property "Reference" "C4"
+		(property "Reference" "C3"
 			(at 100.965 96.52 0)
 			(effects
@@
 			(project "wled_controller"
 				(path "/67a034fd-c582-46b2-83e2-3de9f5f70ac4/07b1b39b-eaae-4ce9-8e52-afae0c59cf87"
-					(reference "C4")
+					(reference "C3")
 					(unit 1)
 				)
@@
 		(dnp no)
 		(fields_autoplaced yes)
-		(property "Reference" "#PWR072"
+		(property "Reference" "#PWR071"
 			(at 109.22 115.57 0)
 			(effects
@@
 			(project "wled_controller"
 				(path "/67a034fd-c582-46b2-83e2-3de9f5f70ac4/07b1b39b-eaae-4ce9-8e52-afae0c59cf87"
-					(reference "#PWR072")
+					(reference "#PWR071")
 					(unit 1)
 				)
@@
 		(on_board yes)
 		(dnp no)
-		(property "Reference" "C7"
+		(property "Reference" "C6"
 			(at 184.15 96.9009 0)
 			(effects
@@
 			(project "wled_controller"
 				(path "/67a034fd-c582-46b2-83e2-3de9f5f70ac4/07b1b39b-eaae-4ce9-8e52-afae0c59cf87"
-					(reference "C7")
+					(reference "C6")
 					(unit 1)
 				)
@@
 		(dnp no)
 		(fields_autoplaced yes)
-		(property "Reference" "#PWR068"
+		(property "Reference" "#PWR067"
 			(at 72.39 115.57 0)
 			(effects
@@
 			(project "wled_controller"
 				(path "/67a034fd-c582-46b2-83e2-3de9f5f70ac4/07b1b39b-eaae-4ce9-8e52-afae0c59cf87"
-					(reference "#PWR068")
+					(reference "#PWR067")
 					(unit 1)
 				)
@@
 		(pin "4"
 		)
-		(pin "1"
+		(pin "2"
 		)
 		(instances
@@
 		(dnp no)
 		(fields_autoplaced yes)
-		(property "Reference" "#PWR073"
+		(property "Reference" "#PWR072"
 			(at 125.73 104.14 0)
 			(effects
@@
 			(project "wled_controller"
 				(path "/67a034fd-c582-46b2-83e2-3de9f5f70ac4/07b1b39b-eaae-4ce9-8e52-afae0c59cf87"
-					(reference "#PWR073")
+					(reference "#PWR072")
 					(unit 1)
 				)
@@
 		(on_board yes)
 		(dnp no)
-		(property "Reference" "#PWR070"
+		(property "Reference" "#PWR069"
 			(at 100.33 86.36 0)
 			(effects
@@
 			(project "wled_controller"
 				(path "/67a034fd-c582-46b2-83e2-3de9f5f70ac4/07b1b39b-eaae-4ce9-8e52-afae0c59cf87"
-					(reference "#PWR070")
+					(reference "#PWR069")
 					(unit 1)
 				)
@@
 		(dnp no)
 		(fields_autoplaced yes)
-		(property "Reference" "#PWR074"
+		(property "Reference" "#PWR073"
 			(at 160.02 115.57 0)
 			(effects
@@
 			(project "wled_controller"
 				(path "/67a034fd-c582-46b2-83e2-3de9f5f70ac4/07b1b39b-eaae-4ce9-8e52-afae0c59cf87"
-					(reference "#PWR074")
-					(unit 1)
-				)
+					(reference "#PWR073")
+					(unit 1)
+				)
