File: hardware/wled_controller/mechanical.kicad_sch (KiCad schematic)
At the start: 9 parts

Commit message: work on pcb
Parts:
- removed H4, H6: MountingHole_Pad, mechanical:MountingHole_3.2mm_M3_DIN965_Pad, symbol Mechanical:MountingHole_Pad
- renumbered H5 to H4
