File: hardware/wled_controller/midi.kicad_sch (KiCad schematic)
At the start: 11 parts, among them J16 DIN-5_180degree, J17 DIN-5_180degree, U7 6N137, U8 74HCT125

Commit message: finalise schematic
Parts:
- R16: Part (none) -> R 10kΩ 125mW 1% 0805
- renumbered J16 to J19, J17 to J20
Connections:
- net +5V: now also U8.13 (EN); no longer U8.1 (EN)
- net MIDI_UART: now also U8.12 (D); no longer U8.2 (D)
- net at R18.1: now also U8.11 (O); no longer U8.3 (O)
Changed lines of the file:
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@@
 		(on_board yes)
 		(dnp no)
-		(property "Reference" "#PWR085"
+		(property "Reference" "#PWR091"
 			(at 187.96 76.2 0)
 			(effects
@@
 			(project "wled_controller"
 				(path "/67a034fd-c582-46b2-83e2-3de9f5f70ac4/8072bd51-fbbd-46ff-a54c-8dc2320b0005"
-					(reference "#PWR085")
+					(reference "#PWR091")
 					(unit 1)
 				)
@@
 		(on_board yes)
 		(dnp no)
-		(property "Reference" "#PWR078"
+		(property "Reference" "#PWR084"
 			(at 100.33 50.8 0)
 			(effects
@@
 			(project "wled_controller"
 				(path "/67a034fd-c582-46b2-83e2-3de9f5f70ac4/8072bd51-fbbd-46ff-a54c-8dc2320b0005"
-					(reference "#PWR078")
+					(reference "#PWR084")
 					(unit 1)
 				)
@@
 		(dnp no)
 		(fields_autoplaced yes)
-		(property "Reference" "#PWR079"
+		(property "Reference" "#PWR085"
 			(at 100.33 66.04 0)
 			(effects
@@
 			(project "wled_controller"
 				(path "/67a034fd-c582-46b2-83e2-3de9f5f70ac4/8072bd51-fbbd-46ff-a54c-8dc2320b0005"
-					(reference "#PWR079")
+					(reference "#PWR085")
 					(unit 1)
 				)
@@
 		(on_board yes)
 		(dnp no)
-		(property "Reference" "#PWR076"
+		(property "Reference" "#PWR082"
 			(at 88.9 50.8 0)
 			(effects
@@
 			(project "wled_controller"
 				(path "/67a034fd-c582-46b2-83e2-3de9f5f70ac4/8072bd51-fbbd-46ff-a54c-8dc2320b0005"
-					(reference "#PWR076")
+					(reference "#PWR082")
 					(unit 1)
 				)
@@
 		(dnp no)
 		(fields_autoplaced yes)
-		(property "Reference" "#PWR089"
+		(property "Reference" "#PWR095"
 			(at 247.65 72.39 0)
 			(effects
@@
 			(project "wled_controller"
 				(path "/67a034fd-c582-46b2-83e2-3de9f5f70ac4/8072bd51-fbbd-46ff-a54c-8dc2320b0005"
-					(reference "#PWR089")
+					(reference "#PWR095")
 					(unit 1)
 				)
@@
 		(dnp no)
 		(fields_autoplaced yes)
-		(property "Reference" "#PWR077"
+		(property "Reference" "#PWR083"
 			(at 88.9 66.04 0)
 			(effects
@@
 			(project "wled_controller"
 				(path "/67a034fd-c582-46b2-83e2-3de9f5f70ac4/8072bd51-fbbd-46ff-a54c-8dc2320b0005"
-					(reference "#PWR077")
+					(reference "#PWR083")
 					(unit 1)
 				)
@@
 		(on_board yes)
 		(dnp no)
-		(property "Reference" "#PWR087"
+		(property "Reference" "#PWR093"
 			(at 209.55 60.96 0)
 			(effects
@@
 			(project "wled_controller"
 				(path "/67a034fd-c582-46b2-83e2-3de9f5f70ac4/8072bd51-fbbd-46ff-a54c-8dc2320b0005"
-					(reference "#PWR087")
+					(reference "#PWR093")
 					(unit 1)
 				)
@@
 		(on_board yes)
 		(dnp no)
-		(property "Reference" "J17"
+		(property "Reference" "J20"
 			(at 237.49 76.2 90)
 			(effects
@@
 			(project ""
 				(path "/67a034fd-c582-46b2-83e2-3de9f5f70ac4/8072bd51-fbbd-46ff-a54c-8dc2320b0005"
-					(reference "J17")
+					(reference "J20")
 					(unit 1)
 				)
@@
 		(on_board yes)
 		(dnp no)
-		(property "Reference" "#PWR080"
+		(property "Reference" "#PWR086"
 			(at 128.27 78.74 0)
 			(effects
@@
 			(project ""
 				(path "/67a034fd-c582-46b2-83e2-3de9f5f70ac4/8072bd51-fbbd-46ff-a54c-8dc2320b0005"
-					(reference "#PWR080")
+					(reference "#PWR086")
 					(unit 1)
 				)
@@
 		(dnp no)
 		(fields_autoplaced yes)
-		(property "Reference" "#PWR088"
+		(property "Reference" "#PWR094"
 			(at 215.9 72.39 0)
 			(effects
@@
 			(project "wled_controller"
 				(path "/67a034fd-c582-46b2-83e2-3de9f5f70ac4/8072bd51-fbbd-46ff-a54c-8dc2320b0005"
-					(reference "#PWR088")
+					(reference "#PWR094")
 					(unit 1)
 				)
@@
 		(on_board yes)
 		(dnp no)
-		(property "Reference" "#PWR083"
+		(property "Reference" "#PWR089"
 			(at 147.32 62.23 0)
 			(effects
@@
 			(project "wled_controller"
 				(path "/67a034fd-c582-46b2-83e2-3de9f5f70ac4/8072bd51-fbbd-46ff-a54c-8dc2320b0005"
-					(reference "#PWR083")
+					(reference "#PWR089")
 					(unit 1)
 				)
@@
 		(on_board yes)
 		(dnp no)
-		(property "Reference" "#PWR082"
+		(property "Reference" "#PWR088"
 			(at 133.35 83.82 0)
 			(effects
@@
 			(project "wled_controller"
 				(path "/67a034fd-c582-46b2-83e2-3de9f5f70ac4/8072bd51-fbbd-46ff-a54c-8dc2320b0005"
-					(reference "#PWR082")
+					(reference "#PWR088")
 					(unit 1)
 				)
@@
 		(on_board yes)
 		(dnp no)
-		(property "Reference" "J16"
+		(property "Reference" "J19"
 			(at 82.55 90.17 90)
 			(effects
@@
 			(project "wled_controller"
 				(path "/67a034fd-c582-46b2-83e2-3de9f5f70ac4/8072bd51-fbbd-46ff-a54c-8dc2320b0005"
-					(reference "J16")
+					(reference "J19")
 					(unit 1)
 				)
@@
 		(lib_id "74xx_IEEE:74125")
 		(at 187.96 83.82 0)
-		(unit 1)
+		(unit 4)
 		(exclude_from_sim no)
 		(in_bom yes)
@@
 				(path "/67a034fd-c582-46b2-83e2-3de9f5f70ac4/8072bd51-fbbd-46ff-a54c-8dc2320b0005"
 					(reference "U8")
-					(unit 1)
+					(unit 4)
 				)
 			)
@@
 			)
 		)
+		(property "Part" "R 10kΩ 125mW 1% 0805"
+			(at 147.32 68.58 0)
+			(effects
+				(font
+					(size 1.27 1.27)
+				)
+				(hide yes)
+			)
+		)
 		(pin "1"
 		)
@@
 		(on_board yes)
 		(dnp no)
-		(property "Reference" "#PWR084"
+		(property "Reference" "#PWR090"
 			(at 177.8 81.28 0)
 			(effects
@@
 			(project "wled_controller"
 				(path "/67a034fd-c582-46b2-83e2-3de9f5f70ac4/8072bd51-fbbd-46ff-a54c-8dc2320b0005"
-					(reference "#PWR084")
+					(reference "#PWR090")
 					(unit 1)
 				)
@@
 		(dnp no)
 		(fields_autoplaced yes)
-		(property "Reference" "#PWR086"
+		(property "Reference" "#PWR092"
 			(at 187.96 104.14 0)
 			(effects
@@
 			(project "wled_controller"
 				(path "/67a034fd-c582-46b2-83e2-3de9f5f70ac4/8072bd51-fbbd-46ff-a54c-8dc2320b0005"
-					(reference "#PWR086")
+					(reference "#PWR092")
 					(unit 1)
 				)
@@
 		(dnp no)
 		(fields_autoplaced yes)
-		(property "Reference" "#PWR081"
+		(property "Reference" "#PWR087"
 			(at 128.27 104.14 0)
 			(effects
@@
 			(project "wled_controller"
 				(path "/67a034fd-c582-46b2-83e2-3de9f5f70ac4/8072bd51-fbbd-46ff-a54c-8dc2320b0005"
-					(reference "#PWR081")
-					(unit 1)
-				)
+					(reference "#PWR087")
+					(unit 1)
+				)

Commit message: some progress on PCB
Parts:
- J19, J20: footprint conn:57PC5F -> conn:DIN5_57PC5F
- U8: renamed from U7; footprint Package_DIP:DIP-8_W7.62mm -> Package_DIP:SMDIP-8_W9.53mm
- renumbered D2 to D3, U8 to U4
Connections:
- net +5V: now also U4.4 (EN); no longer U4.13 (EN)
- net MIDI_UART: now also U4.5 (D); no longer U4.12 (D)
- net at R18.1: now also U4.6 (O); no longer U4.11 (O)
Other:
- moved on the sheet: R16
Changed lines of the file:
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@@
 			)
 		)
-		(property "Footprint" "conn:57PC5F"
+		(property "Footprint" "conn:DIN5_57PC5F"
 			(at 231.14 72.39 0)
 			(effects
@@
 			)
 		)
-		(property "Footprint" "conn:57PC5F"
+		(property "Footprint" "conn:DIN5_57PC5F"
 			(at 76.2 86.36 0)
 			(effects
@@
 		(dnp no)
 		(fields_autoplaced yes)
-		(property "Reference" "U7"
+		(property "Reference" "U8"
 			(at 131.2865 73.66 0)
 			(effects
@@
 			)
 		)
-		(property "Footprint" "Package_DIP:DIP-8_W7.62mm"
+		(property "Footprint" "Package_DIP:SMDIP-8_W9.53mm"
 			(at 128.27 99.06 0)
 			(effects
@@
 			(project ""
 				(path "/67a034fd-c582-46b2-83e2-3de9f5f70ac4/8072bd51-fbbd-46ff-a54c-8dc2320b0005"
-					(reference "U7")
+					(reference "U8")
 					(unit 1)
 				)
@@
 		(lib_id "74xx_IEEE:74125")
 		(at 187.96 83.82 0)
-		(unit 4)
+		(unit 2)
 		(exclude_from_sim no)
 		(in_bom yes)
@@
 		(dnp no)
 		(fields_autoplaced yes)
-		(property "Reference" "U8"
+		(property "Reference" "U4"
 			(at 198.12 77.5014 0)
 			(effects
@@
 			(project "wled_controller"
 				(path "/67a034fd-c582-46b2-83e2-3de9f5f70ac4/8072bd51-fbbd-46ff-a54c-8dc2320b0005"
-					(reference "U8")
-					(unit 4)
+					(reference "U4")
+					(unit 2)
 				)
 			)
@@
 	(symbol
 		(lib_id "Device:R")
-		(at 147.32 68.58 180)
+		(at 147.32 68.58 0)
+		(mirror x)
 		(unit 1)
 		(exclude_from_sim no)
@@
 		(dnp no)
 		(property "Reference" "R16"
-			(at 149.86 66.04 0)
+			(at 144.78 66.04 0)
 			(effects
 				(font
@@
 		)
 		(property "Value" "10kΩ"
-			(at 149.86 68.58 0)
+			(at 144.78 68.58 0)
 			(effects
 				(font
@@
 		)
 		(property "Footprint" "Resistor_SMD:R_0805_2012Metric"
-			(at 149.098 68.58 90)
+			(at 145.542 68.58 90)
 			(effects
 				(font
@@
 		)
 		(property "Info" "125mW 5%"
-			(at 149.86 71.12 0)
+			(at 144.78 71.12 0)
 			(effects
 				(font
@@
 		(dnp no)
 		(fields_autoplaced yes)
-		(property "Reference" "D2"
+		(property "Reference" "D3"
 			(at 113.03 86.3599 90)
 			(effects
@@
 			(project ""
 				(path "/67a034fd-c582-46b2-83e2-3de9f5f70ac4/8072bd51-fbbd-46ff-a54c-8dc2320b0005"
-					(reference "D2")
+					(reference "D3")
 					(unit 1)
 				)

Commit message: work on pcb
Parts:
- removed C12: 100nF, Capacitor_SMD:C_0805_2012Metric, symbol Device:C
- renumbered C11 to C10, R15 to R16, R16 to R17, R17 to R18, R18 to R19

Commit message: update bom
Parts:
- J19, J20: Part 57PC5F -> 0105 05; Shop https://eu.mouser.com/ProductDetail/Switchcraft/57PC5F?qs=M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 -> https://www.tme.eu/be/nl/details/0105-05/din-connectoren/lu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
Changed lines of the file:
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@@
 			)
 		)
-		(property "Part" "57PC5F"
+		(property "Part" "0105 05"
 			(at 231.14 72.39 90)
 			(effects
@@
 			)
 		)
-		(property "Shop" "https://eu.mouser.com/ProductDetail/Switchcraft/57PC5F?qs=MW%252B0w7tSdpkWuZd7MBoFPA%3D%3D"
+		(property "Shop" "https://www.tme.eu/be/nl/details/0105-05/din-connectoren/lumberg/0105-05/"
 			(at 231.14 72.39 90)
 			(effects
@@
 		)
 		(instances
-			(project ""
+			(project "wled_controller"
 				(path "/67a034fd-c582-46b2-83e2-3de9f5f70ac4/8072bd51-fbbd-46ff-a54c-8dc2320b0005"
 					(reference "J20")
@@
 		)
 		(instances
-			(project ""
+			(project "wled_controller"
 				(path "/67a034fd-c582-46b2-83e2-3de9f5f70ac4/8072bd51-fbbd-46ff-a54c-8dc2320b0005"
 					(reference "#PWR084")
@@
 			)
 		)
-		(property "Part" "57PC5F"
+		(property "Part" "0105 05"
 			(at 76.2 86.36 90)
 			(effects
@@
 			)
 		)
-		(property "Shop" "https://eu.mouser.com/ProductDetail/Switchcraft/57PC5F?qs=MW%252B0w7tSdpkWuZd7MBoFPA%3D%3D"
+		(property "Shop" "https://www.tme.eu/be/nl/details/0105-05/din-connectoren/lumberg/0105-05/"
 			(at 76.2 86.36 90)
 			(effects
@@
 		)
 		(instances
-			(project ""
+			(project "wled_controller"
 				(path "/67a034fd-c582-46b2-83e2-3de9f5f70ac4/8072bd51-fbbd-46ff-a54c-8dc2320b0005"
 					(reference "U8")
@@
 		)
 		(instances
-			(project ""
+			(project "wled_controller"
 				(path "/67a034fd-c582-46b2-83e2-3de9f5f70ac4/8072bd51-fbbd-46ff-a54c-8dc2320b0005"
 					(reference "D3")
