File: hardware/wled_controller/usb.kicad_sch (KiCad schematic)
At the start: 5 parts, among them J14 USB_B, J15 Header_01x05, U6 ADUM4160

Commit message: finalise schematic
Parts:
- J17: renamed from J14; Part (none) -> TODO USB_B
- J18: renamed from J15; Part (none) -> Header_01x05
- U6: Part (none) -> ADUM4160BRWZ-RL; Shop (none) -> https://eu.mouser.com/ProductDetail/Analog-Devices/ADUM4160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
Changed lines of the file:
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@@
+			)
+		)
+		(property "Part" " ADUM4160BRWZ-RL"
+			(at 133.35 105.41 0)
+			(effects
+				(font
+					(size 1.27 1.27)
+				)
+				(hide yes)
+			)
+		)
+		(property "Shop" "https://eu.mouser.com/ProductDetail/Analog-Devices/ADUM4160BRWZ-RL?qs=WIvQP4zGaniP0FyiFgFlCw%3D%3D"
+			(at 133.35 105.41 0)
+			(effects
+				(font
+					(size 1.27 1.27)
+				)
+				(hide yes)
 			)
 		)
@@
 		(dnp no)
 		(fields_autoplaced yes)
-		(property "Reference" "#PWR075"
+		(property "Reference" "#PWR081"
 			(at 177.8 120.65 0)
 			(effects
@@
 			(project "wled_controller"
 				(path "/67a034fd-c582-46b2-83e2-3de9f5f70ac4/d13bbfa5-8e48-45fd-ac58-e4bf3e4f5b27"
-					(reference "#PWR075")
+					(reference "#PWR081")
 					(unit 1)
 				)
@@
 		(dnp no)
 		(fields_autoplaced yes)
-		(property "Reference" "#PWR072"
+		(property "Reference" "#PWR078"
 			(at 137.16 129.54 0)
 			(effects
@@
 			(project "wled_controller"
 				(path "/67a034fd-c582-46b2-83e2-3de9f5f70ac4/d13bbfa5-8e48-45fd-ac58-e4bf3e4f5b27"
-					(reference "#PWR072")
+					(reference "#PWR078")
 					(unit 1)
 				)
@@
 		(dnp no)
 		(fields_autoplaced yes)
-		(property "Reference" "#PWR071"
+		(property "Reference" "#PWR077"
 			(at 109.22 96.52 0)
 			(effects
@@
 			(project "wled_controller"
 				(path "/67a034fd-c582-46b2-83e2-3de9f5f70ac4/d13bbfa5-8e48-45fd-ac58-e4bf3e4f5b27"
-					(reference "#PWR071")
+					(reference "#PWR077")
 					(unit 1)
 				)
@@
 		(on_board yes)
 		(dnp no)
-		(property "Reference" "J15"
+		(property "Reference" "J18"
 			(at 184.15 97.79 0)
 			(effects
@@
 			)
 		)
+		(property "Part" "Header_01x05"
+			(at 184.15 102.87 0)
+			(effects
+				(font
+					(size 1.27 1.27)
+				)
+				(hide yes)
+			)
+		)
 		(pin "1"
 		)
@@
 			(project ""
 				(path "/67a034fd-c582-46b2-83e2-3de9f5f70ac4/d13bbfa5-8e48-45fd-ac58-e4bf3e4f5b27"
-					(reference "J15")
+					(reference "J18")
 					(unit 1)
 				)
@@
 		(dnp no)
 		(fields_autoplaced yes)
-		(property "Reference" "#PWR073"
+		(property "Reference" "#PWR079"
 			(at 157.48 96.52 0)
 			(effects
@@
 			(project "wled_controller"
 				(path "/67a034fd-c582-46b2-83e2-3de9f5f70ac4/d13bbfa5-8e48-45fd-ac58-e4bf3e4f5b27"
-					(reference "#PWR073")
+					(reference "#PWR079")
 					(unit 1)
 				)
@@
 		(on_board yes)
 		(dnp no)
-		(property "Reference" "#PWR074"
+		(property "Reference" "#PWR080"
 			(at 175.26 80.01 0)
 			(effects
@@
 			(project ""
 				(path "/67a034fd-c582-46b2-83e2-3de9f5f70ac4/d13bbfa5-8e48-45fd-ac58-e4bf3e4f5b27"
-					(reference "#PWR074")
+					(reference "#PWR080")
 					(unit 1)
 				)
@@
 		(on_board yes)
 		(dnp no)
-		(property "Reference" "J14"
+		(property "Reference" "J17"
 			(at 95.25 87.63 0)
 			(effects
@@
 			)
 		)
+		(property "Part" "TODO USB_B"
+			(at 95.25 100.33 0)
+			(effects
+				(font
+					(size 1.27 1.27)
+				)
+				(hide yes)
+			)
+		)
 		(pin "1"
 		)
@@
 			(project "wled_controller"
 				(path "/67a034fd-c582-46b2-83e2-3de9f5f70ac4/d13bbfa5-8e48-45fd-ac58-e4bf3e4f5b27"
-					(reference "J14")
-					(unit 1)
-				)
+					(reference "J17")
+					(unit 1)
+				)

Commit message: some progress on PCB
Parts:
- J18: Purpose Pin2 D- -> D+; Purpose Pin3 D+ -> D-
- U7: renamed from U6; Part ADUM4160BRWZ-RL -> ADUM4160BRWZ; Shop https://eu.mouser.com/ProductDetail/Analog-Devices/ADUM4160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 -> https://www.tme.eu/bg/details/0105-05/sediniteli-din/lumber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
Connections:
- net GND: no longer C9.2
- net at U7.10 (DD+): now also J18.3 (Pin_3); no longer J18.2 (Pin_2)
- net at U7.11 (DD-): now also J18.2 (Pin_2); no longer J18.3 (Pin_3)
- net at J17.4 (GND), J17.5 (Shield), U7.2 (GND1)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: now also C9.2
Changed lines of the file:
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@@
+	)
+	(junction
+		(at 109.22 121.92)
+		(diameter 0)
+		(color 0 0 0 0)
 	)
 	(junction
@@
 	(wire
 		(pts
+			(xy 165.1 105.41) (xy 167.64 102.87)
+		)
+		(stroke
+			(width 0)
+			(type default)
+		)
+	)
+	(wire
+		(pts
 			(xy 93.98 111.76) (xy 92.71 111.76)
 		)
@@
 	(wire
 		(pts
+			(xy 109.22 121.92) (xy 128.27 121.92)
+		)
+		(stroke
+			(width 0)
+			(type default)
+		)
+	)
+	(wire
+		(pts
 			(xy 149.86 95.25) (xy 149.86 77.47)
 		)
@@
 	(wire
 		(pts
+			(xy 146.05 105.41) (xy 165.1 105.41)
+		)
+		(stroke
+			(width 0)
+			(type default)
+		)
+	)
+	(wire
+		(pts
 			(xy 157.48 87.63) (xy 157.48 90.17)
 		)
@@
 	(wire
 		(pts
-			(xy 146.05 105.41) (xy 179.07 105.41)
+			(xy 167.64 105.41) (xy 165.1 102.87)
 		)
 		(stroke
@@
 	(wire
 		(pts
-			(xy 110.49 105.41) (xy 110.49 102.87)
+			(xy 111.76 105.41) (xy 111.76 102.87)
 		)
 		(stroke
@@
 	(wire
 		(pts
-			(xy 120.65 105.41) (xy 110.49 105.41)
+			(xy 120.65 105.41) (xy 111.76 105.41)
 		)
 		(stroke
@@
 	(wire
 		(pts
-			(xy 102.87 100.33) (xy 113.03 100.33)
-		)
-		(stroke
-			(width 0)
-			(type default)
-		)
-	)
-	(wire
-		(pts
-			(xy 113.03 102.87) (xy 120.65 102.87)
+			(xy 102.87 100.33) (xy 114.3 100.33)
+		)
+		(stroke
+			(width 0)
+			(type default)
+		)
+	)
+	(wire
+		(pts
+			(xy 114.3 102.87) (xy 120.65 102.87)
 		)
 		(stroke
@@
 	(wire
 		(pts
-			(xy 110.49 102.87) (xy 102.87 102.87)
+			(xy 111.76 102.87) (xy 102.87 102.87)
 		)
 		(stroke
@@
 	(wire
 		(pts
+			(xy 167.64 102.87) (xy 179.07 102.87)
+		)
+		(stroke
+			(width 0)
+			(type default)
+		)
+	)
+	(wire
+		(pts
 			(xy 157.48 77.47) (xy 157.48 80.01)
 		)
@@
 	(wire
 		(pts
-			(xy 113.03 100.33) (xy 113.03 102.87)
+			(xy 146.05 102.87) (xy 165.1 102.87)
+		)
+		(stroke
+			(width 0)
+			(type default)
+		)
+	)
+	(wire
+		(pts
+			(xy 114.3 100.33) (xy 114.3 102.87)
 		)
 		(stroke
@@
 	(wire
 		(pts
-			(xy 146.05 102.87) (xy 179.07 102.87)
-		)
-		(stroke
-			(width 0)
-			(type default)
-		)
-	)
-	(wire
-		(pts
 			(xy 179.07 100.33) (xy 175.26 100.33)
 		)
@@
 	(wire
 		(pts
-			(xy 109.22 87.63) (xy 109.22 90.17)
+			(xy 109.22 87.63) (xy 109.22 121.92)
+		)
+		(stroke
+			(width 0)
+			(type default)
+		)
+	)
+	(wire
+		(pts
+			(xy 179.07 105.41) (xy 167.64 105.41)
 		)
 		(stroke
@@
 	(wire
 		(pts
-			(xy 93.98 121.92) (xy 128.27 121.92)
+			(xy 93.98 121.92) (xy 109.22 121.92)
 		)
 		(stroke
@@
 		(dnp no)
 		(fields_autoplaced yes)
-		(property "Reference" "U6"
+		(property "Reference" "U7"
 			(at 138.0841 87.63 0)
 			(effects
@@
 			)
 		)
-		(property "Part" " ADUM4160BRWZ-RL"
+		(property "Part" "ADUM4160BRWZ"
 			(at 133.35 105.41 0)
 			(effects
@@
 			)
 		)
-		(property "Shop" "https://eu.mouser.com/ProductDetail/Analog-Devices/ADUM4160BRWZ-RL?qs=WIvQP4zGaniP0FyiFgFlCw%3D%3D"
+		(property "Shop" "https://www.tme.eu/bg/details/0105-05/sediniteli-din/lumberg/0105-05/"
 			(at 133.35 105.41 0)
 			(effects
@@
 			(project "wled_controller"
 				(path "/67a034fd-c582-46b2-83e2-3de9f5f70ac4/d13bbfa5-8e48-45fd-ac58-e4bf3e4f5b27"
-					(reference "U6")
+					(reference "U7")
 					(unit 1)
 				)
@@
 	)
 	(symbol
-		(lib_id "power:GND")
-		(at 109.22 90.17 0)
-		(unit 1)
-		(exclude_from_sim no)
-		(in_bom yes)
-		(on_board yes)
-		(dnp no)
-		(fields_autoplaced yes)
-		(property "Reference" "#PWR077"
-			(at 109.22 96.52 0)
-			(effects
-				(font
-					(size 1.27 1.27)
-				)
-				(hide yes)
-			)
-		)
-		(property "Value" "GND"
-			(at 109.22 95.25 0)
-			(effects
-				(font
-					(size 1.27 1.27)
-				)
-				(hide yes)
-			)
-		)
-		(property "Footprint" ""
-			(at 109.22 90.17 0)
-			(effects
-				(font
-					(size 1.27 1.27)
-				)
-				(hide yes)
-			)
-		)
-		(property "Datasheet" ""
-			(at 109.22 90.17 0)
-			(effects
-				(font
-					(size 1.27 1.27)
-				)
-				(hide yes)
-			)
-		)
-		(property "Description" ""
-			(at 109.22 90.17 0)
-			(effects
-				(font
-					(size 1.27 1.27)
-				)
-				(hide yes)
-			)
-		)
-		(pin "1"
-		)
-		(instances
-			(project "wled_controller"
-				(path "/67a034fd-c582-46b2-83e2-3de9f5f70ac4/d13bbfa5-8e48-45fd-ac58-e4bf3e4f5b27"
-					(reference "#PWR077")
-					(unit 1)
-				)
-			)
-		)
-	)
-	(symbol
 		(lib_id "conn:Conn_01x05")
 		(at 184.15 102.87 0)
@@
 			)
 		)
-		(property "Purpose Pin2" "D-"
+		(property "Purpose Pin2" "D+"
 			(at 184.15 105.41 0)
 			(do_not_autoplace yes)
@@
 			)
 		)
-		(property "Purpose Pin3" "D+"
+		(property "Purpose Pin3" "D-"
 			(at 184.15 102.87 0)
 			(do_not_autoplace yes)

Commit message: work on pcb
Parts:
- added R15: 10kΩ, Resistor_SMD:R_0805_2012Metric, symbol Device:R
- J17: Part TODO USB_B -> 61729-0010BLF; Shop (none) -> https://eu.mouser.com/ProductDetail/Amphenol-FCI/61729-0010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
- renumbered C9 to C8, C10 to C9
Connections:
- net USB_EN: now also R15.1
- new net +3.3V: R15.2

Commit message: update bom
Parts:
- U7: Shop https://www.tme.eu/bg/details/0105-05/sediniteli-din/lumber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 -> https://www.tme.eu/be/nl/details/adum4160brwz/geint-schakel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
Changed lines of the file:
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@@
 			)
 		)
-		(property "Shop" "https://www.tme.eu/bg/details/0105-05/sediniteli-din/lumberg/0105-05/"
+		(property "Shop" "https://www.tme.eu/be/nl/details/adum4160brwz/geint-schakelingen-overige-interfaces/analog-devices/"
 			(at 133.35 105.41 0)
 			(effects
@@
 		)
 		(instances
-			(project ""
+			(project "wled_controller"
 				(path "/67a034fd-c582-46b2-83e2-3de9f5f70ac4/d13bbfa5-8e48-45fd-ac58-e4bf3e4f5b27"
 					(reference "J18")
@@
 		)
 		(instances
-			(project ""
+			(project "wled_controller"
 				(path "/67a034fd-c582-46b2-83e2-3de9f5f70ac4/d13bbfa5-8e48-45fd-ac58-e4bf3e4f5b27"
 					(reference "#PWR078")
@@
 			)
 		)
-		(property "Datasheet" " ~"
+		(property "Datasheet" "~"
 			(at 99.06 101.6 0)
 			(effects
