File: hardware/wled_controller/wled_controller.kicad_sch (KiCad schematic)
At the start: 5 parts, among them U1 Pico

Commit message: finalise schematic
Parts:
- D1: Part (none) -> SK34A
- U1: footprint RPi_Pico:RPi_Pico_SMD_TH -> MCU_RaspberryPi_and_Boards:RPi_Pico_TH; Part (none) -> 2x Header_01x20
Connections:
- net DEN: now also U1.27 (GPIO21); no longer U1.26 (GPIO20)
- net USB_EN: now also U1.29 (GPIO22); no longer U1.24 (GPIO18)
- net D14: now reaches U1.25 (GPIO19)
- new net D13: U1.24 (GPIO18)
- new net D15: U1.26 (GPIO20)
- no-connect marks 11 -> 8
Other:
- sheet Drivers ports: added D13, D14, D15; removed none
Changed lines of the file:
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@@
-	)
-	(no_connect
-		(at 146.05 104.14)
 	)
 	(no_connect
@@
 	)
 	(no_connect
-		(at 146.05 109.22)
-	)
-	(no_connect
 		(at 110.49 83.82)
 	)
@@
 	)
 	(no_connect
-		(at 146.05 114.3)
-	)
-	(no_connect
 		(at 146.05 76.2)
 	)
@@
 	(wire
 		(pts
+			(xy 199.39 118.11) (xy 209.55 118.11)
+		)
+		(stroke
+			(width 0)
+			(type default)
+		)
+	)
+	(wire
+		(pts
+			(xy 199.39 113.03) (xy 209.55 113.03)
+		)
+		(stroke
+			(width 0)
+			(type default)
+		)
+	)
+	(wire
+		(pts
 			(xy 153.67 121.92) (xy 146.05 121.92)
 		)
@@
 	(wire
 		(pts
+			(xy 156.21 116.84) (xy 146.05 116.84)
+		)
+		(stroke
+			(width 0)
+			(type default)
+		)
+	)
+	(wire
+		(pts
 			(xy 149.86 78.74) (xy 146.05 78.74)
 		)
@@
 	(wire
 		(pts
+			(xy 156.21 109.22) (xy 146.05 109.22)
+		)
+		(stroke
+			(width 0)
+			(type default)
+		)
+	)
+	(wire
+		(pts
+			(xy 110.49 106.68) (xy 109.22 106.68)
+		)
+		(stroke
+			(width 0)
+			(type default)
+		)
+	)
+	(wire
+		(pts
+			(xy 199.39 82.55) (xy 209.55 82.55)
+		)
+		(stroke
+			(width 0)
+			(type default)
+		)
+	)
+	(wire
+		(pts
+			(xy 95.25 69.85) (xy 95.25 78.74)
+		)
+		(stroke
+			(width 0)
+			(type default)
+		)
+	)
+	(wire
+		(pts
+			(xy 146.05 119.38) (xy 147.32 119.38)
+		)
+		(stroke
+			(width 0)
+			(type default)
+		)
+	)
+	(wire
+		(pts
+			(xy 152.4 74.93) (xy 152.4 78.74)
+		)
+		(stroke
+			(width 0)
+			(type default)
+		)
+	)
+	(wire
+		(pts
 			(xy 156.21 111.76) (xy 146.05 111.76)
 		)
@@
 	(wire
 		(pts
-			(xy 110.49 106.68) (xy 109.22 106.68)
-		)
-		(stroke
-			(width 0)
-			(type default)
-		)
-	)
-	(wire
-		(pts
-			(xy 199.39 82.55) (xy 209.55 82.55)
-		)
-		(stroke
-			(width 0)
-			(type default)
-		)
-	)
-	(wire
-		(pts
-			(xy 95.25 69.85) (xy 95.25 78.74)
-		)
-		(stroke
-			(width 0)
-			(type default)
-		)
-	)
-	(wire
-		(pts
-			(xy 146.05 119.38) (xy 147.32 119.38)
-		)
-		(stroke
-			(width 0)
-			(type default)
-		)
-	)
-	(wire
-		(pts
-			(xy 152.4 74.93) (xy 152.4 78.74)
-		)
-		(stroke
-			(width 0)
-			(type default)
-		)
-	)
-	(wire
-		(pts
 			(xy 146.05 81.28) (xy 147.32 81.28)
 		)
@@
 	(wire
 		(pts
-			(xy 156.21 116.84) (xy 146.05 116.84)
+			(xy 199.39 115.57) (xy 209.55 115.57)
+		)
+		(stroke
+			(width 0)
+			(type default)
+		)
+	)
+	(wire
+		(pts
+			(xy 156.21 104.14) (xy 146.05 104.14)
 		)
 		(stroke
@@
 	(wire
 		(pts
-			(xy 199.39 125.73) (xy 209.55 125.73)
+			(xy 199.39 130.81) (xy 209.55 130.81)
 		)
 		(stroke
@@
 		(pts
 			(xy 102.87 121.92) (xy 110.49 121.92)
+		)
+		(stroke
+			(width 0)
+			(type default)
+		)
+	)
+	(wire
+		(pts
+			(xy 156.21 114.3) (xy 146.05 114.3)
 		)
 		(stroke
@@
 	)
 	(label "USB_EN"
-		(at 199.39 125.73 0)
+		(at 199.39 130.81 0)
 		(fields_autoplaced yes)
 		(effects
@@
 	)
 	(label "USB_EN"
+		(at 156.21 104.14 180)
+		(fields_autoplaced yes)
+		(effects
+			(font
+				(size 1.27 1.27)
+			)
+			(justify right bottom)
+		)
+	)
+	(label "D13"
 		(at 156.21 116.84 180)
 		(fields_autoplaced yes)
@@
 		)
 	)
+	(label "D13"
+		(at 199.39 113.03 0)
+		(fields_autoplaced yes)
+		(effects
+			(font
+				(size 1.27 1.27)
+			)
+			(justify left bottom)
+		)
+	)
 	(label "D10"
 		(at 199.39 105.41 0)
@@
 		)
 	)
+	(label "D14"
+		(at 199.39 115.57 0)
+		(fields_autoplaced yes)
+		(effects
+			(font
+				(size 1.27 1.27)
+			)
+			(justify left bottom)
+		)
+	)
 	(label "D11"
 		(at 199.39 107.95 0)
@@
 	)
 	(label "DEN"
-		(at 156.21 111.76 180)
+		(at 156.21 109.22 180)
+		(fields_autoplaced yes)
+		(effects
+			(font
+				(size 1.27 1.27)
+			)
+			(justify right bottom)
+		)
+	)
+	(label "D15"
+		(at 199.39 118.11 0)
+		(fields_autoplaced yes)
+		(effects
+			(font
+				(size 1.27 1.27)
+			)
+			(justify left bottom)
+		)
+	)
+	(label "D14"
+		(at 156.21 114.3 180)
 		(fields_autoplaced yes)
 		(effects
@@
 			)
 			(justify left bottom)
+		)
+	)
+	(label "D15"
+		(at 156.21 111.76 180)
+		(fields_autoplaced yes)
+		(effects
+			(font
+				(size 1.27 1.27)
+			)
+			(justify right bottom)
 		)
 	)
@@
 		(property "Shop" "https://store.comet.bg/Catalogue/Product/49266/"
 			(at 152.4 71.12 90)
+			(effects
+				(font
+					(size 1.27 1.27)
+				)
+				(hide yes)
+			)
+		)
+		(property "Part" "SK34A"
+			(at 152.4 71.12 0)
 			(effects
 				(font
@@
 			)
 		)
-		(property "Footprint" "RPi_Pico:RPi_Pico_SMD_TH"
+		(property "Footprint" "MCU_RaspberryPi_and_Boards:RPi_Pico_TH"
 			(at 128.27 100.33 90)
 			(effects
@@
 		)
 		(property "Description" ""
+			(at 128.27 100.33 0)
+			(effects
+				(font
+					(size 1.27 1.27)
+				)
+				(hide yes)
+			)
+		)
+		(property "Part" "2x Header_01x20"
 			(at 128.27 100.33 0)
 			(effects
@@
 	(sheet
 		(at 209.55 76.2)
-		(size 25.4 36.83)
+		(size 25.4 43.18)
 		(fields_autoplaced yes)
 		(stroke
@@
 		)
 		(property "Sheetfile" "drivers.kicad_sch"
-			(at 209.55 113.6146 0)
+			(at 209.55 119.9646 0)
 			(effects
 				(font
@@
 		(pin "DEN" input
 			(at 209.55 80.01 180)
+			(effects
+				(font
+					(size 1.27 1.27)
+				)
+				(justify left)
+			)
+		)
+		(pin "D13" input
+			(at 209.55 113.03 180)
+			(effects
+				(font
+					(size 1.27 1.27)
+				)
+				(justify left)
+			)
+		)
+		(pin "D14" input
+			(at 209.55 115.57 180)
+			(effects
+				(font
+					(size 1.27 1.27)
+				)
+				(justify left)
+			)
+		)
+		(pin "D15" input
+			(at 209.55 118.11 180)
 			(effects
 				(font
@@
 	)
 	(sheet
-		(at 209.55 123.19)
-		(size 25.4 10.16)
+		(at 209.55 128.27)
+		(size 25.4 5.08)
 		(fields_autoplaced yes)
 		(stroke
@@
 		)
 		(property "Sheetname" "USB"
-			(at 209.55 122.4784 0)
+			(at 209.55 127.5584 0)
 			(effects
 				(font
@@
 		)
 		(pin "USB_EN" input
-			(at 209.55 125.73 180)
-			(effects
-				(font
+			(at 209.55 130.81 180)
+			(effects
+				(font

Commit message: some progress on PCB
Parts:
- removed C3: 100nF, Capacitor_SMD:C_0805_2012Metric, symbol Device:C
Connections:
- net DMX512/DIR: now also U1.4 (GPIO2); no longer U1.5 (GPIO3)
- net DMX512/RX: now also U1.1 (GPIO0); no longer U1.6 (GPIO4)
- net DMX512/TX: now also U1.2 (GPIO1); no longer U1.7 (GPIO5)
- net MIDI/MIDI_UART: now also U1.7 (GPIO5); no longer U1.2 (GPIO1)
Other:
- added sheet Mechanical (mechanical.kicad_sch)
Changed lines of the file:
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@@
-	)
-	(no_connect
-		(at 110.49 76.2)
 	)
 	(no_connect
@@
 	)
 	(no_connect
-		(at 110.49 83.82)
+		(at 146.05 99.06)
 	)
 	(no_connect
-		(at 146.05 99.06)
+		(at 110.49 86.36)
+	)
+	(no_connect
+		(at 110.49 88.9)
 	)
 	(no_connect
@@
 	(wire
 		(pts
-			(xy 163.83 86.36) (xy 163.83 87.63)
-		)
-		(stroke
-			(width 0)
-			(type default)
-		)
-	)
-	(wire
-		(pts
 			(xy 199.39 92.71) (xy 209.55 92.71)
 		)
@@
 	(wire
 		(pts
+			(xy 97.79 81.28) (xy 86.36 81.28)
+		)
+		(stroke
+			(width 0)
+			(type default)
+		)
+	)
+	(wire
+		(pts
 			(xy 199.39 118.11) (xy 209.55 118.11)
 		)
@@
 	(wire
 		(pts
-			(xy 90.17 88.9) (xy 110.49 88.9)
+			(xy 97.79 83.82) (xy 97.79 81.28)
 		)
 		(stroke
@@
 	(wire
 		(pts
-			(xy 90.17 69.85) (xy 95.25 69.85)
-		)
-		(stroke
-			(width 0)
-			(type default)
-		)
-	)
-	(wire
-		(pts
-			(xy 163.83 95.25) (xy 163.83 99.06)
-		)
-		(stroke
-			(width 0)
-			(type default)
-		)
-	)
-	(wire
-		(pts
 			(xy 163.83 86.36) (xy 168.91 86.36)
 		)
@@
 	(wire
 		(pts
-			(xy 95.25 69.85) (xy 95.25 78.74)
-		)
-		(stroke
-			(width 0)
-			(type default)
-		)
-	)
-	(wire
-		(pts
 			(xy 146.05 119.38) (xy 147.32 119.38)
 		)
@@
 	(wire
 		(pts
-			(xy 95.25 78.74) (xy 110.49 78.74)
-		)
-		(stroke
-			(width 0)
-			(type default)
-		)
-	)
-	(wire
-		(pts
-			(xy 90.17 91.44) (xy 110.49 91.44)
+			(xy 86.36 91.44) (xy 110.49 91.44)
 		)
 		(stroke
@@
 	(wire
 		(pts
+			(xy 86.36 76.2) (xy 110.49 76.2)
+		)
+		(stroke
+			(width 0)
+			(type default)
+		)
+	)
+	(wire
+		(pts
 			(xy 199.39 110.49) (xy 209.55 110.49)
 		)
@@
 	(wire
 		(pts
+			(xy 110.49 83.82) (xy 97.79 83.82)
+		)
+		(stroke
+			(width 0)
+			(type default)
+		)
+	)
+	(wire
+		(pts
 			(xy 149.86 77.47) (xy 149.86 78.74)
 		)
@@
 	(wire
 		(pts
-			(xy 90.17 86.36) (xy 110.49 86.36)
+			(xy 86.36 78.74) (xy 110.49 78.74)
 		)
 		(stroke
@@
 				(path "/67a034fd-c582-46b2-83e2-3de9f5f70ac4"
 					(reference "#PWR012")
-					(unit 1)
-				)
-			)
-		)
-	)
-	(symbol
-		(lib_id "Device:C")
-		(at 163.83 91.44 0)
-		(unit 1)
-		(exclude_from_sim no)
-		(in_bom yes)
-		(on_board yes)
-		(dnp no)
-		(property "Reference" "C3"
-			(at 163.83 88.9 0)
-			(effects
-				(font
-					(size 1.27 1.27)
-				)
-				(justify left)
-			)
-		)
-		(property "Value" "100nF"
-			(at 163.83 96.52 0)
-			(effects
-				(font
-					(size 1.27 1.27)
-				)
-				(justify left)
-			)
-		)
-		(property "Footprint" "Capacitor_SMD:C_0805_2012Metric"
-			(at 164.7952 95.25 0)
-			(effects
-				(font
-					(size 1.27 1.27)
-				)
-				(hide yes)
-			)
-		)
-		(property "Datasheet" "~"
-			(at 163.83 91.44 0)
-			(effects
-				(font
-					(size 1.27 1.27)
-				)
-				(hide yes)
-			)
-		)
-		(property "Description" ""
-			(at 163.83 91.44 0)
-			(effects
-				(font
-					(size 1.27 1.27)
-				)
-				(hide yes)
-			)
-		)
-		(property "Info" "16V"
-			(at 163.83 93.98 0)
-			(effects
-				(font
-					(size 1.27 1.27)
-				)
-				(justify left)
-			)
-		)
-		(property "Shop" "https://store.comet.bg/Catalogue/Product/16789/"
-			(at 163.83 91.44 0)
-			(effects
-				(font
-					(size 1.27 1.27)
-				)
-				(hide yes)
-			)
-		)
-		(property "Part" "C 100nF 16V 0805"
-			(at 163.83 91.44 0)
-			(effects
-				(font
-					(size 1.27 1.27)
-				)
-				(hide yes)
-			)
-		)
-		(pin "1"
-		)
-		(pin "2"
-		)
-		(instances
-			(project "wled_controller"
-				(path "/67a034fd-c582-46b2-83e2-3de9f5f70ac4"
-					(reference "C3")
 					(unit 1)
 				)
@@
 	(symbol
 		(lib_id "power:GND")
-		(at 163.83 99.06 0)
-		(unit 1)
-		(exclude_from_sim no)
-		(in_bom yes)
-		(on_board yes)
-		(dnp no)
-		(fields_autoplaced yes)
-		(property "Reference" "#PWR010"
-			(at 163.83 105.41 0)
-			(effects
-				(font
-					(size 1.27 1.27)
-				)
-				(hide yes)
-			)
-		)
-		(property "Value" "GND"
-			(at 163.83 104.14 0)
-			(effects
-				(font
-					(size 1.27 1.27)
-				)
-				(hide yes)
-			)
-		)
-		(property "Footprint" ""
-			(at 163.83 99.06 0)
-			(effects
-				(font
-					(size 1.27 1.27)
-				)
-				(hide yes)
-			)
-		)
-		(property "Datasheet" ""
-			(at 163.83 99.06 0)
-			(effects
-				(font
-					(size 1.27 1.27)
-				)
-				(hide yes)
-			)
-		)
-		(property "Description" ""
-			(at 163.83 99.06 0)
-			(effects
-				(font
-					(size 1.27 1.27)
-				)
-				(hide yes)
-			)
-		)
-		(pin "1"
-		)
-		(instances
-			(project "wled_controller"
-				(path "/67a034fd-c582-46b2-83e2-3de9f5f70ac4"
-					(reference "#PWR010")
-					(unit 1)
-				)
-			)
-		)
-	)
-	(symbol
-		(lib_id "power:GND")
 		(at 109.22 81.28 270)
 		(unit 1)
@@
 	(sheet
 		(at 209.55 76.2)
-		(size 25.4 43.18)
+		(size 25.4 45.72)
 		(fields_autoplaced yes)
 		(stroke
@@
 		)
 		(property "Sheetfile" "drivers.kicad_sch"
-			(at 209.55 119.9646 0)
+			(at 209.55 122.5046 0)
 			(effects
 				(font
@@
 	)
 	(sheet
-		(at 63.5 67.31)
+		(at 59.69 88.9)
 		(size 26.67 5.08)
 		(fields_autoplaced yes)
@@
 		)
 		(property "Sheetname" "MIDI"
-			(at 63.5 66.5984 0)
+			(at 59.69 88.1884 0)
 			(effects
 				(font
@@
 		)
 		(property "Sheetfile" "midi.kicad_sch"
-			(at 63.5 72.9746 0)
+			(at 59.69 94.5646 0)
 			(effects
 				(font
@@
 		)
 		(pin "MIDI_UART" output
-			(at 90.17 69.85 0)
+			(at 86.36 91.44 0)
 			(effects
 				(font
@@
 	)
 	(sheet
+		(at 63.5 143.51)
+		(size 26.67 10.16)
+		(fields_autoplaced yes)
+		(stroke
+			(width 0.1524)
+			(type solid)
+		)
+		(fill
+			(color 0 0 0 0.0000)
+		)
+		(property "Sheetname" "Mechanical"
+			(at 63.5 142.7984 0)
+			(effects
+				(font
+					(size 1.27 1.27)
+				)
+				(justify left bottom)
+			)
+		)
+		(property "Sheetfile" "mechanical.kicad_sch"
+			(at 63.5 154.2546 0)
+			(effects
+				(font
+					(size 1.27 1.27)
+				)
+				(justify left top)
+			)
+		)
+		(instances
+			(project "wled_controller"
+				(path "/67a034fd-c582-46b2-83e2-3de9f5f70ac4"
+					(page "22")
+				)
+			)
+		)
+	)
+	(sheet
 		(at 209.55 128.27)
 		(size 25.4 5.08)
@@
 	)
 	(sheet
-		(at 63.5 83.82)
+		(at 59.69 73.66)
 		(size 26.67 10.16)
-		(fields_autoplaced yes)
 		(stroke
 			(width 0.1524)
@@
 		)
 		(property "Sheetname" "DMX512"
-			(at 63.5 83.1084 0)
+			(at 59.69 73.66 0)
 			(effects
 				(font
@@
 		)
 		(property "Sheetfile" "dmx512.kicad_sch"
-			(at 63.5 94.5646 0)
+			(at 59.69 84.4046 0)
 			(effects
 				(font
@@
 		)
 		(pin "RX" input
-			(at 90.17 88.9 0)
+			(at 86.36 76.2 0)
 			(effects
 				(font
@@
 		)
 		(pin "DIR" input
-			(at 90.17 86.36 0)
+			(at 86.36 81.28 0)
 			(effects
 				(font
@@
 		)
 		(pin "TX" output
-			(at 90.17 91.44 0)
-			(effects
-				(font
+			(at 86.36 78.74 0)
+			(effects
+				(font

Commit message: work on pcb
Connections:
- net D1: now also U1.20 (GPIO15); no longer U1.9 (GPIO6)
- net D10: now also U1.26 (GPIO20); no longer U1.20 (GPIO15)
- net D11: now also U1.9 (GPIO6); no longer U1.21 (GPIO16)
- net D12: now also U1.24 (GPIO18); no longer U1.22 (GPIO17)
- net D13: now also U1.25 (GPIO19); no longer U1.24 (GPIO18)
- net D14: now also U1.22 (GPIO17); no longer U1.25 (GPIO19)
- net D15: now also U1.21 (GPIO16); no longer U1.26 (GPIO20)
- net D2: now also U1.19 (GPIO14); no longer U1.10 (GPIO7)
- net D3: now also U1.17 (GPIO13); no longer U1.11 (GPIO8)
- net D4: now also U1.16 (GPIO12); no longer U1.12 (GPIO9)
- net D5: now also U1.15 (GPIO11); no longer U1.14 (GPIO10)
- net D6: now also U1.12 (GPIO9); no longer U1.15 (GPIO11)
- net D7: now also U1.14 (GPIO10); no longer U1.16 (GPIO12)
- net D8: now also U1.11 (GPIO8); no longer U1.17 (GPIO13)
- net D9: now also U1.10 (GPIO7); no longer U1.19 (GPIO14)
Changed lines of the file:
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@@
 	(wire
 		(pts
-			(xy 153.67 121.92) (xy 146.05 121.92)
+			(xy 156.21 121.92) (xy 146.05 121.92)
 		)
 		(stroke
@@
 	(wire
 		(pts
-			(xy 153.67 124.46) (xy 146.05 124.46)
+			(xy 156.21 124.46) (xy 146.05 124.46)
 		)
 		(stroke
@@
 	)
 	(label "D11"
-		(at 153.67 124.46 180)
-		(fields_autoplaced yes)
-		(effects
-			(font
-				(size 1.27 1.27)
-			)
-			(justify right bottom)
+		(at 102.87 96.52 0)
+		(fields_autoplaced yes)
+		(effects
+			(font
+				(size 1.27 1.27)
+			)
+			(justify left bottom)
 		)
 	)
@@
 	)
 	(label "D13"
-		(at 156.21 116.84 180)
+		(at 156.21 114.3 180)
 		(fields_autoplaced yes)
 		(effects
@@
 	)
 	(label "D7"
-		(at 102.87 114.3 0)
+		(at 102.87 109.22 0)
 		(fields_autoplaced yes)
 		(effects
@@
 	)
 	(label "D9"
-		(at 102.87 121.92 0)
+		(at 102.87 99.06 0)
 		(fields_autoplaced yes)
 		(effects
@@
 	)
 	(label "D8"
-		(at 102.87 116.84 0)
+		(at 102.87 101.6 0)
 		(fields_autoplaced yes)
 		(effects
@@
 	)
 	(label "D14"
-		(at 156.21 114.3 180)
+		(at 156.21 121.92 180)
 		(fields_autoplaced yes)
 		(effects
@@
 	)
 	(label "D2"
-		(at 102.87 99.06 0)
+		(at 102.87 121.92 0)
 		(fields_autoplaced yes)
 		(effects
@@
 	)
 	(label "D1"
-		(at 102.87 96.52 0)
+		(at 102.87 124.46 0)
 		(fields_autoplaced yes)
 		(effects
@@
 	)
 	(label "D3"
-		(at 102.87 101.6 0)
+		(at 102.87 116.84 0)
 		(fields_autoplaced yes)
 		(effects
@@
 	)
 	(label "D5"
-		(at 102.87 109.22 0)
+		(at 102.87 111.76 0)
 		(fields_autoplaced yes)
 		(effects
@@
 	)
 	(label "D15"
-		(at 156.21 111.76 180)
+		(at 156.21 124.46 180)
 		(fields_autoplaced yes)
 		(effects
@@
 	)
 	(label "D12"
-		(at 153.67 121.92 180)
+		(at 156.21 116.84 180)
 		(fields_autoplaced yes)
 		(effects
@@
 	)
 	(label "D10"
-		(at 102.87 124.46 0)
-		(fields_autoplaced yes)
-		(effects
-			(font
-				(size 1.27 1.27)
-			)
-			(justify left bottom)
+		(at 156.21 111.76 180)
+		(fields_autoplaced yes)
+		(effects
+			(font
+				(size 1.27 1.27)
+			)
+			(justify right bottom)
 		)
 	)
@@
 	)
 	(label "D4"
-		(at 102.87 104.14 0)
+		(at 102.87 114.3 0)
 		(fields_autoplaced yes)
 		(effects
@@
 	)
 	(label "D6"
-		(at 102.87 111.76 0)
+		(at 102.87 104.14 0)
 		(fields_autoplaced yes)
 		(effects
@@
 		(dnp no)
 		(fields_autoplaced yes)
-		(property "Reference" "#PWR011"
+		(property "Reference" "#PWR010"
 			(at 172.72 63.5 0)
 			(effects
@@
 			(project "wled_controller"
 				(path "/67a034fd-c582-46b2-83e2-3de9f5f70ac4"
-					(reference "#PWR011")
+					(reference "#PWR010")
 					(unit 1)
 				)
@@
 		(dnp no)
 		(fields_autoplaced yes)
-		(property "Reference" "#PWR012"
+		(property "Reference" "#PWR011"
 			(at 172.72 78.74 0)
 			(effects
@@
 			(project "wled_controller"
 				(path "/67a034fd-c582-46b2-83e2-3de9f5f70ac4"
-					(reference "#PWR012")
+					(reference "#PWR011")
 					(unit 1)
 				)
@@
 		(on_board yes)
 		(dnp no)
-		(property "Reference" "#PWR013"
+		(property "Reference" "#PWR012"
 			(at 165.1 86.36 0)
 			(effects
@@
 			(project ""
 				(path "/67a034fd-c582-46b2-83e2-3de9f5f70ac4"
-					(reference "#PWR013")
+					(reference "#PWR012")
 					(unit 1)
 				)
